File: 8086_add_latch_buffers.sch (KiCad schematic (older format))
At the start: 23 parts

Commit message: updating 8086 design
Parts:
- removed C? (x5): 104, symbol C
- removed U? (x4): 74LS08, symbol 74LS08
- removed U?: 74LS04, symbol 74LS04
- removed U?: 74LS244, symbol 74LS244
- gave numbers to parts that had none: 12
Connections:
- net BUSRQ: now reaches U24.1 (OE)
- net BUSRQ: now also U21.19 (CE), U22.19 (CE), U23.19 (CE), U25.1 (OE), U26.1 (OE)
- net ~RD renamed WR/~RD
- no-connect marks 0 -> 18
Other:
- note removed: "R/W SIGNAL DECODING"
- moved on the sheet: C29, C30, C31, C32, C33, C34, U21, U22, U23, U24, U25, U26
