File: 8086_decoding.sch (KiCad schematic (older format))
At the start: 12 parts

Commit message: updating 8086 design
Parts:
- added unit 3 of U10
- added U32: 74LS08, symbol 74LS08
- gave numbers to parts that had none: 10
Connections:
- net +5V: now also U10.14 (VCC), U32.14 (VCC)
- net A15: now also U10.5
- net A16: now also U10.9; no longer U10.5
- net GND: now also U30.4 (E1), U10.7 (GND), U32.7 (GND)
- net ~A15: now also U10.6
- net ~IORD: now also U32.2
- net ~IOWR: now also U32.1
- net ~RAM_SEL: now also U10.10; no longer U10.8
- net at U34.1: now also U10.8; no longer U10.6
- net M/~IO renamed ~IOSEL
- net ~IOSEL: now also U32.3
- net ~ROM_SEL: no longer names the net of U33.6, U34.2, U34.5
- net ~ROM_SEL: now also U10.11; no longer U10.9
- no-connect marks 0 -> 15
Other:
- moved on the sheet: C39, C40, C41, C42, C43, U33A
