File: 8086_ram.sch (KiCad schematic (older format))
At the start: 10 parts

Commit message: updating 8086 design
Parts:
- removed C? (x4): 104, symbol C
- added R1: 2.2k, symbol R
- added RN2, RN3: 2.2k, Resistors_THT:R_Array_SIP9, symbol R_Network08
- added SW2, SW3: SW_DIP_x08, symbol SW_DIP_x08
- added U11, U12: 74LS299, symbol 74LS299
- gave numbers to parts that had none: 6
Connections:
- net VCC is gone; now on net +5V: U10.14 (VCC)
- net +5V: now also R1.1, SW2.10, SW2.11, SW2.12, SW2.13, SW2.14, SW2.15, SW2.16, SW2.9, SW3.10, SW3.11, SW3.12, SW3.13, SW3.14, SW3.15, SW3.16, SW3.9, U11.1 (S0), U11.20 (VCC), U11.9 (Mr), U12.1 (S0), U12.20 (VCC), U12.9 (Mr)
- net 8207_WE: now also U10.1; no longer U10.11
- net GND: now also RN2.1 (common), RN3.1 (common), U11.10 (GND), U11.2 (OE1), U11.3 (OE2), U12.10 (GND), U12.2 (OE1), U12.3 (OE2)
- net ~8207_WE: now also U10.2; no longer U10.10
- net ~RAM_SEL: now also U9.67 (~PEA); no longer U9.10 (CE)
- net PCLK: now reaches U9.12 (MUX/PCLK)
- net PCLK: now also U11.12 (Cp), U12.12 (Cp)
- net 8207_RESET: now reaches U9.17 (RESET)
- net 8207_RESET: now also U11.19 (S1), U12.19 (S1)
- net ~AACKA: now reaches U9.4 (~AACKA~/~WZ)
- net PDI: now reaches U9.57 (PDI)
- net PDI: now also U12.17 (Q7)
- net at U9.58 (RFRQ): now also R1.2
- net 86_CLOCK: now reaches U9.59 (CLK)
- net ~S1: now reaches U9.65 (~RDA)
- net ~S0: now reaches U9.66 (~WRA)
- net ~S2: now reaches U9.68 (PCTLA)
- new net: U11.17 (Q7), U12.11 (Ds0)
- new net: RN3.3 (R2), SW3.2, U12.13 (IO1)
- new net: RN3.5 (R4), SW3.4, U12.14 (IO3)
- new net: RN3.7 (R6), SW3.6, U12.15 (IO5)
- new net: RN3.9 (R8), SW3.8, U12.16 (IO7)
- new net: RN3.8 (R7), SW3.7, U12.4 (IO6)
- new net: RN3.6 (R5), SW3.5, U12.5 (IO4)
- new net: RN3.4 (R3), SW3.3, U12.6 (IO2)
- new net: RN3.2 (R1), SW3.1, U12.7 (IO0)
- new net: RN2.3 (R2), SW2.2, U11.13 (IO1)
- new net: RN2.5 (R4), SW2.4, U11.14 (IO3)
- new net: RN2.7 (R6), SW2.6, U11.15 (IO5)
- new net: RN2.9 (R8), SW2.8, U11.16 (IO7)
- new net: RN2.8 (R7), SW2.7, U11.4 (IO6)
- new net: RN2.6 (R5), SW2.5, U11.5 (IO4)
- new net: RN2.4 (R3), SW2.3, U11.6 (IO2)
- new net: RN2.2 (R1), SW2.1, U11.7 (IO0)
- no-connect marks 0 -> 21
Other:
- note added: "8207 PROGRAM DATA WORD"
- note added: "Port Select Out\nA/~B"
- moved on the sheet: C10, C11, C12, C9, U9
