File: 8086_rom.sch (KiCad schematic (older format))
At the start: 9 parts

Commit message: updating 8086 design
Parts:
- removed C? (x5): 104, symbol C
- added C5, C6, C7, C8: 104, symbol C
- gave numbers to parts that had none: 4
Connections:
- net +5V: now also C5.1, C6.1, C7.1, C8.1
- net GND: now also C5.2, C6.2, C7.2, C8.2
