File: 8086_sbc.sch (KiCad schematic (older format))
At the start: 10 parts

Commit message: updating 8086 design
Parts:
- removed C?: 104, symbol C
- removed U?: 8086_Min_Mode, Housings_DIP:DIP-40_W15.24mm, symbol 8086_Min_Mode
- removed U?: DS1813, symbol DS1813
- added RN1: 2.2k, Resistors_THT:R_Array_SIP9, symbol R_Network08
- added U2: 8086_Max_Mode, Housings_DIP:DIP-40_W15.24mm, symbol 8086_Max_Mode
- added U3: 8288, Housings_DIP:DIP-20_W7.62mm, symbol 8288
- added U4: ATTINY45-20PU, Housings_DIP:DIP-8_W7.62mm, symbol ATTINY45-20PU
- SW1: renamed from SW?; value SW_Push -> SW_RESET
- gave numbers to parts that had none: 6
Connections:
- net +5V: now also U1.18 (VCC), U2.40 (VCC), U3.15 (CEN), U3.20 (VCC), U4.8 (VCC)
- net /RESET: now also U4.6 (PB1(MISO/DO/AIN1/OC0B/OC1A/PCINT1)); no longer SW1.1
- net A16/S3: now also U2.38 (A16/S3)
- net A17/S4: now also U2.37 (A17/S4)
- net A18/S5: now also U2.36 (A18/S5)
- net A19/S6: now also U2.35 (A19/S6)
- net AD0: now also U2.16 (AD0)
- net AD1: now also U2.15 (AD1)
- net AD10: now also U2.6 (AD10)
- net AD11: now also U2.5 (AD11)
- net AD12: now also U2.4 (AD12)
- net AD13: now also U2.3 (AD13)
- net AD14: now also U2.2 (AD14)
- net AD15: now also U2.39 (AD15)
- net AD2: now also U2.14 (AD2)
- net AD3: now also U2.13 (AD3)
- net AD4: now also U2.12 (AD4)
- net AD5: now also U2.11 (AD5)
- net AD6: now also U2.10 (AD6)
- net AD7: now also U2.9 (AD7)
- net AD8: now also U2.8 (AD8)
- net AD9: now also U2.7 (AD9)
- net ALE: now also U3.5 (ALE)
- net CLOCK: now also RN1.9 (R8)
- net DT/~R: now also U3.4 (DT/~R~)
- net GND: now also RN1.1 (common), U2.1 (GND), U2.20 (GND), U2.33 (MN/~MX~), U3.1 (IOB), U3.10 (GND), U3.6 (~AEN~), U4.4 (GND)
- net INT: now also RN1.3 (R2), U2.18 (INTR)
- net NMI: now also RN1.2 (R1), U2.17 (NMI)
- net PCLOCK: now also RN1.8 (R7)
- net READY2: now also RN1.6 (R5)
- net ~BHE/S7: now also U2.34 (~BHE~/S7)
- net ~DEN: now also U3.16 (DEN)
- net ~INTA: now also U3.14 (~INTA~)
- net ~IORD: now also U3.13 (~IORC~)
- net ~IOWR: now also U3.11 (~IOWC~)
- net ~MEMRD: now also U3.7 (~MRDC~)
- net ~MEMWR: now also U3.9 (~MWTC~)
- net ~TEST: now also RN1.5 (R4), U2.23 (~TEST~)
- net 86_CLOCK: now reaches U1.8 (CLK)
- net 86_CLOCK: now also U2.19 (CLK), U3.2 (CLK)
- net at U1.10 (RESET): now also U2.21 (RESET)
- net at U1.5 (READY): now also U2.22 (READY)
- net READY1 renamed ~AACKA
- new net: SW1.1, U4.1 (PB5(~RESET~/dW/ADC0/PCINT5))
- new net 8207_RESET: U4.5 (PB0(MOSI/DI/SDA/AIN0/OC0A/OC1A/AREF/PCINT0))
- new net BUSRQ: RN1.4 (R3)
- new net MCE/~PDEN: U3.17 (MCE/~PDEN~)
- new net WR/~RD: U2.32 (~RD~)
- new net ~AIOWC: U3.12 (~AIOWC~)
- new net ~AMWC: U3.8 (~AMWC~)
- new net ~S0: U2.26 (~S0~), U3.19 (~S0~)
- new net ~S1: U2.27 (~S1~), U3.3 (~S1~)
- new net ~S2: U2.28 (~S2~), U3.18 (~S2~)
- no-connect marks 0 -> 15
Other:
- note added: "SYSTEM\nBUS\nMODE"
- moved on the sheet: C1, C2, C3, C4, SW1, U1, Y1
