File: 8086_simm.sch (KiCad schematic (older format))
At the start: 24 parts

Commit message: updating 8086 design
Parts:
- gave numbers to parts that had none: 24
Connections:
- no-connect marks 24 -> 48
Other:
- moved on the sheet: C13, C14, C15, C16, C17, C18, C19, C20, C21, C22, C23, C24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
